File: pcb/e3tp3pcb/e3tp3pcb.kicad_pcb (KiCad board)
At the start: 2 copper layers, 96.5 x 96.5 mm, 52 parts, among them J1 Conn_01x06_Female, J10 Left, J11 USB_B, J13 Conn_01x02_Male, J14 Conn_01x02_Female, J15 Right, J2 Conn_01x04_Female, J3 Conn_01x05_Female, J4 Conn_01x08_Male, J5 supplyKeyboard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

Commit message: suma, resta, negativos, cociente, encadenación
Co-authored-by: Matias Alvarez <matalvarez62275@users.noreply.github.com>
Routing:
- net (no net): track 0.00 -> 3.21 mm
Changed lines of the file:
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@@
     (effects (font (size 1 1) (thickness 0.15)))
   )
+  (segment (start 232.755 67.655) (end 233.68 67.655) (width 0.25) (layer "B.Cu") (net 0))
+  (segment (start 231.14 66.04) (end 232.755 67.655) (width 0.25) (layer "B.Cu") (net 0))
   (segment (start 182.88 100.33) (end 188.595 100.33) (width 1) (layer "B.Cu") (net 4))
   (segment (start 191.77 97.155) (end 194.36 97.155) (width 1) (layer "B.Cu") (net 4))

Commit message: pos fixes pcb kicad
Parts:
- added R10: 10k, Resistor_SMD:R_0805_2012Metric, B.Cu at (141.5, 100.3)
- added R11: 10k, Resistor_SMD:R_0805_2012Metric, B.Cu at (141.5, 97.8)
- added R12: 10k, Resistor_SMD:R_0805_2012Metric, B.Cu at (141.5, 102.9)
- added R8: 10k, Resistor_SMD:R_0805_2012Metric, B.Cu at (141.4, 105.4)
- added R9: 10k, Resistor_SMD:R_0805_2012Metric, B.Cu at (141.5, 95.2)
- moved C3 72.6 mm to (188.8, 53.5)
- moved C10 72.6 mm to (111.5, 131.4)
- moved C14 72.6 mm to (117.1, 135.8)
- moved C15 72.6 mm to (124.0, 51.4)
- moved C4 72.6 mm to (127.8, 135.8)
- moved C5 72.6 mm to (158.8, 110.4)
- moved J10 72.6 mm to (126.6, 130.8)
- moved J13 72.6 mm to (198.9, 119.4)
- moved SW4 72.6 mm to (180.6, 96.9)
- moved SW6 72.6 mm to (162.8, 126.1)
- moved C1 72.6 mm to (148.9, 110.4)
- moved C11 72.6 mm to (194.6, 53.2)
- moved C12 72.6 mm to (131.9, 115.4)
- moved C16 72.6 mm to (135.7, 111.4)
- moved C2 72.6 mm to (124.5, 135.8)
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Connections:
- net /IOB_4A renamed /C2
- net /IOB_8A renamed /C0
- net /IOB_9B renamed /C1
- J1 pad 1: /FLASH_MISO -> /IOB_20A
Routing:
- net GND: track 551.0 -> 626.0 mm
- net +3V3: track 63.4 -> 105.3 mm, vias 0 -> 2
- net /FLASH_MISO: track 12.8 -> 0.00 mm
- net /IOB_20A: track 20.4 -> 33.2 mm
- net (no net): track 3.21 -> 0.00 mm
- net /IOT_37A: track 39.1 -> 41.1 mm
- net /IOT_39A: track 47.7 -> 49.6 mm
- net /IOT_43A: track 16.3 -> 18.3 mm
- net /IOT_36B: track 23.0 -> 25.0 mm
- net /IOT_38B: track 32.0 -> 33.9 mm
Other:
- board text added: "22.13 - Electrónica 3 - TP2 Grupo 3 2022 ITBA"
- board text removed: "22.13 - Electrónica 3 - TP2 Grupo 1 2022 ITBA"
