File: pcb/e3tp3pcb/e3tp3pcb.kicad_sch (KiCad schematic)
At the start: 52 parts, among them J1 Conn_01x06_Female, J10 Left, J11 USB_B, J13 Conn_01x02_Male, J14 Conn_01x02_Female, J15 Right, J2 Conn_01x04_Female, J3 Conn_01x05_Female, J4 Conn_01x08_Male, J5 supplyKeyboard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

Commit message: pos fixes pcb kicad
Parts:
- added R10, R11, R12, R8, R9: 10k, Resistor_SMD:R_0805_2012Metric, symbol Device:R
Connections:
- net +3V3: now also R10.2, R11.2, R12.2, R8.2, R9.2
- net FLASH_MISO: no longer J1.1 (Pin_1)
- net IOB_20A: now also J1.1 (Pin_1)
- net IOT_36B: now also R12.1
- net IOT_37A: now also R8.1
- net IOT_38B: now also R11.1
- net IOT_39A: now also R10.1
- net IOT_43A: now also R9.1
Other:
- company: (none) -> 22.13 - Electrónica III - Grupo 03
- title: (none) -> TP N° 2: Implementación de calculadora en FPGA
- moved on the sheet: SW1, SW2, SW3, SW4, SW5
